Commit message: remove hardcoded paths

File: go2/go2.urdf (robot description, URDF)
Before this commit: robot go2, 13 links, 12 joints
Links:
- link FL_calf: geometry collision cylinder length=0.065 radius=0.011; collision cylinder length=0.12 radius=0.012
- link FL_hip: geometry collision cylinder length=0.092 radius=0.02; visual mesh filename=./assets/hip_0.obj scale=1 1 1
- link FL_thigh: geometry collision box size=0.034 0.0245 0.213; visual mesh filename=./assets/thigh_0.obj scale=1 1 1
- link FR_calf: geometry collision cylinder length=0.065 radius=0.011; collision cylinder length=0.12 radius=0.013
- link FR_hip: geometry collision cylinder length=0.092 radius=0.02; visual mesh filename=./assets/hip_0.obj scale=1 1 1
- link FR_thigh: geometry collision box size=0.034 0.0245 0.213; visual mesh filename=./assets/thigh_mirror_0.obj scale=1 1 1
- link RL_calf: geometry collision cylinder length=0.065 radius=0.011; collision cylinder length=0.12 radius=0.013
- link RL_hip: geometry collision cylinder length=0.092 radius=0.02; visual mesh filename=./assets/hip_0.obj scale=1 1 1
- link RL_thigh: geometry collision box size=0.034 0.0245 0.213; visual mesh filename=./assets/thigh_0.obj scale=1 1 1
- link RR_calf: geometry collision cylinder length=0.065 radius=0.011; collision cylinder length=0.12 radius=0.013
- link RR_hip: geometry collision cylinder length=0.092 radius=0.02; visual mesh filename=./assets/hip_0.obj scale=1 1 1
- link RR_thigh: geometry collision box size=0.034 0.0245 0.213; visual mesh filename=./assets/thigh_mirror_0.obj scale=1 1 1
- link base_link: geometry collision box size=0.3762 0.0935 0.114; collision cylinder length=0.09 radius=0.05
